File: breadboard_ne555/breadboard_ne555.sch (KiCad schematic (older format))
At the start: 12 parts, among them J1 USB_B_Micro, J2 Conn_02x02_Odd_Even, J3 Conn_02x02_Odd_Even, J4 Conn_01x05, U1 NE555

Commit message: update: change package 0603 to 0805
Parts:
- C1, C3: footprint Capacitor_SMD:C_0603_1608Metric_Pad1.05x0.95mm_HandSolder -> digikey-footprints:0805
- R1, R2: footprint Resistor_SMD:R_0603_1608Metric_Pad1.05x0.95mm_HandSolder -> digikey-footprints:0805
Changed lines of the file:
@@
 F 0 "R1" H 6670 3596 50  0000 L CNN
 F 1 "300" H 6670 3505 50  0000 L CNN
-F 2 "Resistor_SMD:R_0603_1608Metric_Pad1.05x0.95mm_HandSolder" V 6530 3550 50  0001 C CNN
+F 2 "digikey-footprints:0805" V 6530 3550 50  0001 C CNN
 F 3 "~" H 6600 3550 50  0001 C CNN
 	1    6600 3550
@@
 F 0 "C1" H 4100 3700 50  0000 L CNN
 F 1 "104" H 4100 3500 50  0000 L CNN
-F 2 "Capacitor_SMD:C_0603_1608Metric_Pad1.05x0.95mm_HandSolder" H 4088 3450 50  0001 C CNN
+F 2 "digikey-footprints:0805" H 4088 3450 50  0001 C CNN
 F 3 "~" H 4050 3600 50  0001 C CNN
 	1    4050 3600
@@
 F 0 "C3" H 4815 3996 50  0000 L CNN
 F 1 "103" H 4815 3905 50  0000 L CNN
-F 2 "Capacitor_SMD:C_0603_1608Metric_Pad1.05x0.95mm_HandSolder" H 4738 3800 50  0001 C CNN
+F 2 "digikey-footprints:0805" H 4738 3800 50  0001 C CNN
 F 3 "~" H 4700 3950 50  0001 C CNN
 	1    4700 3950
@@
 F 0 "R2" V 5950 3350 50  0000 L CNN
 F 1 "1K" V 6050 3350 50  0000 L CNN
-F 2 "Resistor_SMD:R_0603_1608Metric_Pad1.05x0.95mm_HandSolder" V 5980 3400 50  0001 C CNN
+F 2 "digikey-footprints:0805" V 5980 3400 50  0001 C CNN
 F 3 "~" H 6050 3400 50  0001 C CNN
 	1    6050 3400

Commit message: update change to pcb
Parts:
- D1: footprint LED_SMD:LED_0805_2012Metric -> digikey-footprints:0805
Changed lines of the file:
@@
 F 0 "D1" V 6650 3825 50  0000 R CNN
 F 1 "LED" V 6550 3825 50  0000 R CNN
-F 2 "LED_SMD:LED_0805_2012Metric" H 6600 3900 50  0001 C CNN
+F 2 "digikey-footprints:0805" H 6600 3900 50  0001 C CNN
 F 3 "~" H 6600 3900 50  0001 C CNN
 	1    6600 3900
